Commit message: removed warnings

File: aida_env/urdf/aida.urdf (robot description, URDF)
Before this commit: robot aida, 33 links, 32 joints
Links:
- link asus_camera_link: mass None -> 0
- link asus_camera_link_optical: mass None -> 0
- link base_laser: mass None -> 0
- link base_link: mass None -> 0
- link nav_module_link: mass None -> 0
- link rgb_cam_rl_link: mass None -> 0
- link rgb_cam_rr_link: mass None -> 0

Commit message: fixed no gravity

File: aida_env/urdf/aida.urdf (robot description, URDF)
Before this commit: robot aida, 33 links, 32 joints
Links:
- link base_link: mass 0 -> None

Commit message: Changed lots of parameters

File: aida_env/urdf/aida.urdf (robot description, URDF)
Before this commit: robot aida, 33 links, 32 joints
Joints:
- joint left_front_foot_hinge: origin xyz=0.3 0 0 rpy=0 0 0 -> xyz=0.3 0 0.1 rpy=0 0 0
- joint left_rear_foot_hinge: origin xyz=0.3 0 0 rpy=0 0 0 -> xyz=0.3 0 0.1 rpy=0 0 0
- joint right_front_foot_hinge: origin xyz=0.3 0 0 rpy=0 0 0 -> xyz=0.3 0 0.1 rpy=0 0 0
- joint right_rear_foot_hinge: origin xyz=0.3 0 0 rpy=0 0 0 -> xyz=0.3 0 0.1 rpy=0 0 0
